File: V3/rj45-breakout-8ch-v3.kicad_sch (KiCad schematic)
At the start: 16 parts, among them J1 Jack RJ45, J10 DB141V-2.54-6P, J11 DB141V-2.54-6P, J12 DB141V-2.54-6P, J13 DB141V-2.54-6P, J2 Jack RJ45, J3 Jack RJ45, J4 Jack RJ45, J5 Jack RJ45, J6 Jack RJ45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

Commit message: Replaced 2.54mm pitch terminal blocks for 3.5mm pitch.
Parts:
- J10, J11, J12, J13: value DB141V-2.54-6P -> 250-206; footprint Tales:TerminalBlock_Dibo_DB141V-2.54-6P_1x06_P2.54mm_Vertical -> Tales:TerminalBlock_Wago_250-206_1x06_P3.5mm_45Degree; LCSC Part C2898748 -> C2765065; Mfr DIBO -> Wago; Mfr PN DB141V-2.54-6P -> 250-206; Vendor PN C2898748 -> C2765065
- J9: value DB142V-5.08-2P -> 250-202; footprint Tales:TerminalBlock_Dibo_DB142V-5.08-2P_1x02_P5.08mm_Vertical -> Tales:TerminalBlock_Wago_250-202_1x02_P3.5mm_45Degree; LCSC Part C2898699 -> C2765061; Mfr DIBO -> Wago; Mfr PN DB142V-5.08-2P -> 250-202; Vendor PN C2898699 -> C2765061
Other:
- title: 8 Channel RJ45 Breakout Board -> eumesmo 8 Channel RJ45 Breakout Board
