File: V3/eumesmo-brk-8ch-v3.kicad_pcb (KiCad board)
At the start: 2 copper layers, 103 x 67.8 mm, 17 parts, among them J1 Jack RJ45, J10 250-206, J11 250-206, J12 250-206, J13 250-206, J2 Jack RJ45, J3 Jack RJ45, J4 Jack RJ45, J5 Jack RJ45, J6 Jack RJ45, J7 Jack RJ45, J8 Jack RJ45, J9 250-202

Commit message: Revised Metaltex holders
Other:
- board text added: "SUPORTES PCI METALTEX SP7 1x pé macho 9 mm 1x pé fêmea 9 mm 1x espaçador 45 mm 2x espaçador 20 mm Comprimento total 103 mm Largura da placa 67,8 mm"
- board text removed: "SUPORTES PCI METALTEX SP7 1x pé macho 9 mm 1x pé fêmea 9 mm 1x espaçador 45 mm 1x espaçador 30 mm 1x espaçador 10 mm Comprimento total 103 mm Largura da placa 67,8 mm"
Changed lines of the file:
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@@
 		)
 	)
-	(gr_text "SUPORTES PCI METALTEX SP7\n1x pé macho  9 mm\n1x pé fêmea 9 mm\n1x espaçador 45 mm\n1x espaçador 30 mm\n1x espaçador 10 mm\nComprimento total 103 mm\nLargura da placa 67,8 mm"
+	(gr_text "SUPORTES PCI METALTEX SP7\n1x pé macho  9 mm\n1x pé fêmea 9 mm\n1x espaçador 45 mm\n2x espaçador 20 mm\nComprimento total 103 mm\nLargura da placa 67,8 mm"
 		(at 100 132 0)
 		(layer "Cmts.User")
@@
 		(layer "Dwgs.User")
 		(pts
-			(xy 100 62.219592) (xy 204.999999 62.219592)
+			(xy 100 62.219592) (xy 203 62.219592)
 		)
 		(height -4.219592)
@@
 			(keep_text_aligned yes)
 		)
-		(gr_text "105.0000 mm"
-			(at 152.5 56.85 0)
+		(gr_text "103.0000 mm"
+			(at 151.5 56.85 0)
 			(layer "Dwgs.User")
 			(effects
