File: V3/eumesmo-brk-8ch-v3.kicad_pcb (KiCad board)
At the start: 2 copper layers, 103 x 67.8 mm, 17 parts, among them J1 Jack RJ45, J10 250-206, J11 250-206, J12 250-206, J13 250-206, J2 Jack RJ45, J3 Jack RJ45, J4 Jack RJ45, J5 Jack RJ45, J6 Jack RJ45, J7 Jack RJ45, J8 Jack RJ45, J9 250-202

Commit message: Adjusted component rotation and offset information for JLCPCB.
Parts:
- moved G*** 1.52 mm to (107.5, 76.8)
Other:
- board text added: "V3.1 2026-09-12"
- board text removed: "V3.1 2026-06-17"

Commit message: Adjusted comment regarding DIN rail modules.
Other:
- board text added: "SUPORTES PCI METALTEX SP7 MÓDULO EUMESMO-BRK-8CH-V3 1x pé macho 9 mm 1x pé fêmea 9 mm 1x espaçador 45 mm 2x espaçador 20 mm Comprimento total 103 mm Largura da placa 67,8 mm"
- board text removed: "SUPORTES PCI METALTEX SP7 1x pé macho 9 mm 1x pé fêmea 9 mm 1x espaçador 45 mm 2x espaçador 20 mm Comprimento total 103 mm Largura da placa 67,8 mm"
Changed lines of the file:
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@@
 		)
 	)
-	(gr_text "SUPORTES PCI METALTEX SP7\n1x pé macho  9 mm\n1x pé fêmea 9 mm\n1x espaçador 45 mm\n2x espaçador 20 mm\nComprimento total 103 mm\nLargura da placa 67,8 mm"
+	(gr_text "SUPORTES PCI METALTEX SP7\nMÓDULO EUMESMO-BRK-8CH-V3\n1x pé macho  9 mm\n1x pé fêmea 9 mm\n1x espaçador 45 mm\n2x espaçador 20 mm\nComprimento total 103 mm\nLargura da placa 67,8 mm"
 		(at 100 132 0)
 		(layer "Cmts.User")

Commit message: Adjusted terminal blocks positions
Parts:
- moved J10 1.00 mm to (122.0, 118.0)
- moved J11 1.00 mm to (145.0, 118.0)
- moved J12 1.00 mm to (168.0, 118.0)
- moved J13 1.00 mm to (191.0, 118.0)
- moved J9 1.00 mm to (106.0, 118.0)
Routing:
- net /CH8PAR4: track 54.9 -> 53.9 mm
- net /CH5PAR4: track 26.8 -> 25.8 mm
- net /CH1PAR4: track 26.4 -> 25.4 mm
- net /CH8PAR3: track 49.6 -> 48.6 mm
- net /CH8PAR2: track 56.2 -> 55.2 mm
- net /CH7PAR3: track 31.5 -> 30.5 mm
- net /CH7PAR2: track 27.7 -> 26.7 mm
- net /CH6PAR3: track 49.4 -> 48.4 mm
- net /CH6PAR2: track 56.2 -> 55.2 mm
- net /CH5PAR3: track 31.3 -> 30.3 mm
- net /CH5PAR2: track 27.9 -> 26.9 mm
- net /CH4PAR3: track 49.2 -> 48.2 mm
- net /CH4PAR2: track 56.4 -> 55.4 mm
- net /CH3PAR4: track 26.6 -> 25.6 mm
- net /CH3PAR3: track 31.4 -> 30.4 mm
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Other:
- board text added: "V3.1 2026-09-23"
- board text removed: "V3.1 2026-09-12"
