File: V3/eumesmo-brk-8ch-v3.kicad_sch (KiCad schematic)
At the start: 16 parts, among them J1 Jack RJ45, J10 250-206, J11 250-206, J12 250-206, J13 250-206, J2 Jack RJ45, J3 Jack RJ45, J4 Jack RJ45, J5 Jack RJ45, J6 Jack RJ45, J7 Jack RJ45, J8 Jack RJ45, J9 250-202

Commit message: Adjusted component rotation and offset information for JLCPCB.
Parts:
- J1, J2, J3, J4, J5, J6, J7, J8: FT Position Offset (none) -> 0,3.609; FT Rotation Offset (none) -> 0; JLCPCB BOM 1 -> (none); LCSC Part C2902702 -> (none); LCSC Part # (none) -> C2902702
- J10, J11, J12, J13: FT Position Offset (none) -> 0,0; FT Rotation Offset (none) -> 0; JLCPCB BOM 1 -> (none); LCSC Part C2765065 -> (none); LCSC Part # (none) -> C2765065
- J9: FT Position Offset (none) -> 0,0; FT Rotation Offset (none) -> 0; JLCPCB BOM 1 -> (none); LCSC Part C2765061 -> (none); LCSC Part # (none) -> C2765061

Commit message: Adjusted components offset
Parts:
- J10, J11, J12, J13, J9: FT Position Offset 0,0 -> (none)
Changed lines of the file:
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@@
 			)
 		)
-		(property "FT Position Offset" "0,0"
+		(property "FT Position Offset" ""
 			(at 218.44 64.77 0)
 			(hide yes)
@@
 			)
 		)
-		(property "FT Position Offset" "0,0"
+		(property "FT Position Offset" ""
 			(at 119.38 125.73 0)
 			(hide yes)
@@
 			)
 		)
-		(property "FT Position Offset" "0,0"
+		(property "FT Position Offset" ""
 			(at 113.03 29.21 0)
 			(hide yes)
@@
 			)
 		)
-		(property "FT Position Offset" "0,0"
+		(property "FT Position Offset" ""
 			(at 119.38 64.77 0)
 			(hide yes)
@@
 			)
 		)
-		(property "FT Position Offset" "0,0"
+		(property "FT Position Offset" ""
 			(at 218.44 125.73 0)
 			(hide yes)

Commit message: Replaced Wago connectors for other brand, no stock.
Parts:
- J10, J11, J12, J13: LCSC Part # C2765065 -> C475158; Mfr Wago -> Cixi Kefa Elec; Mfr PN 250-206 -> KF250-3.5-6P-1; Vendor PN C2765065 -> C475158
- J9: LCSC Part # C2765061 -> C475154; Mfr Wago -> Cixi Kefa Elec; Mfr PN 250-202 -> KF250-3.5-2P-1; Vendor PN C2765061 -> C475154
Changed lines of the file:
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@@
 			)
 		)
-		(property "Mfr" "Wago"
+		(property "Mfr" "Cixi Kefa Elec"
 			(at 218.44 64.77 0)
 			(hide yes)
@@
 			)
 		)
-		(property "Mfr PN" "250-206"
+		(property "Mfr PN" "KF250-3.5-6P-1"
 			(at 218.44 64.77 0)
 			(hide yes)
@@
 			)
 		)
-		(property "Vendor PN" "C2765065"
+		(property "Vendor PN" "C475158"
 			(at 218.44 64.77 0)
 			(hide yes)
@@
 			)
 		)
-		(property "LCSC Part #" "C2765065"
+		(property "LCSC Part #" "C475158"
 			(at 218.44 64.77 0)
 			(hide yes)
@@
 			)
 		)
-		(property "Mfr" "Wago"
-			(at 119.38 125.73 0)
-			(hide yes)
-			(show_name no)
-			(do_not_autoplace no)
-			(effects
-				(font
-					(size 1.27 1.27)
-				)
-			)
-		)
-		(property "Mfr PN" "250-206"
+		(property "Mfr" "Cixi Kefa Elec"
+			(at 119.38 125.73 0)
+			(hide yes)
+			(show_name no)
+			(do_not_autoplace no)
+			(effects
+				(font
+					(size 1.27 1.27)
+				)
+			)
+		)
+		(property "Mfr PN" "KF250-3.5-6P-1"
 			(at 119.38 125.73 0)
 			(hide yes)
@@
 			)
 		)
-		(property "Vendor PN" "C2765065"
+		(property "Vendor PN" "C475158"
 			(at 119.38 125.73 0)
 			(hide yes)
@@
 			)
 		)
-		(property "LCSC Part #" "C2765065"
+		(property "LCSC Part #" "C475158"
 			(at 119.38 125.73 0)
 			(hide yes)
@@
 			)
 		)
-		(property "Mfr" "Wago"
-			(at 113.03 29.21 0)
-			(hide yes)
-			(show_name no)
-			(do_not_autoplace no)
-			(effects
-				(font
-					(size 1.27 1.27)
-				)
-			)
-		)
-		(property "Mfr PN" "250-202"
+		(property "Mfr" "Cixi Kefa Elec"
+			(at 113.03 29.21 0)
+			(hide yes)
+			(show_name no)
+			(do_not_autoplace no)
+			(effects
+				(font
+					(size 1.27 1.27)
+				)
+			)
+		)
+		(property "Mfr PN" "KF250-3.5-2P-1"
 			(at 113.03 29.21 0)
 			(hide yes)
@@
 			)
 		)
-		(property "Vendor PN" "C2765061"
+		(property "Vendor PN" "C475154"
 			(at 113.03 29.21 0)
 			(hide yes)
@@
 			)
 		)
-		(property "LCSC Part #" "C2765061"
+		(property "LCSC Part #" "C475154"
 			(at 113.03 29.21 0)
 			(hide yes)
@@
 			)
 		)
-		(property "Mfr" "Wago"
-			(at 119.38 64.77 0)
-			(hide yes)
-			(show_name no)
-			(do_not_autoplace no)
-			(effects
-				(font
-					(size 1.27 1.27)
-				)
-			)
-		)
-		(property "Mfr PN" "250-206"
+		(property "Mfr" "Cixi Kefa Elec"
+			(at 119.38 64.77 0)
+			(hide yes)
+			(show_name no)
+			(do_not_autoplace no)
+			(effects
+				(font
+					(size 1.27 1.27)
+				)
+			)
+		)
+		(property "Mfr PN" "KF250-3.5-6P-1"
 			(at 119.38 64.77 0)
 			(hide yes)
@@
 			)
 		)
-		(property "Vendor PN" "C2765065"
+		(property "Vendor PN" "C475158"
 			(at 119.38 64.77 0)
 			(hide yes)
@@
 			)
 		)
-		(property "LCSC Part #" "C2765065"
+		(property "LCSC Part #" "C475158"
 			(at 119.38 64.77 0)
 			(hide yes)
@@
 			)
 		)
-		(property "Mfr" "Wago"
-			(at 218.44 125.73 0)
-			(hide yes)
-			(show_name no)
-			(do_not_autoplace no)
-			(effects
-				(font
-					(size 1.27 1.27)
-				)
-			)
-		)
-		(property "Mfr PN" "250-206"
+		(property "Mfr" "Cixi Kefa Elec"
+			(at 218.44 125.73 0)
+			(hide yes)
+			(show_name no)
+			(do_not_autoplace no)
+			(effects
+				(font
+					(size 1.27 1.27)
+				)
+			)
+		)
+		(property "Mfr PN" "KF250-3.5-6P-1"
 			(at 218.44 125.73 0)
 			(hide yes)
@@
 			)
 		)
-		(property "Vendor PN" "C2765065"
+		(property "Vendor PN" "C475158"
 			(at 218.44 125.73 0)
 			(hide yes)
@@
 			)
 		)
-		(property "LCSC Part #" "C2765065"
-			(at 218.44 125.73 0)
-			(hide yes)
+		(property "LCSC Part #" "C475158"
+			(at 218.44 125.73 0)
+			(hide yes)
